File: BM71-Dongle.kicad_pcb (KiCad board)
At the start: 2 copper layers, 12 x 17 mm, 11 parts, among them J1 USB_B_Micro, SW1 SW, SW2 SW, U1 BM71, U2 NJM12877F33

Commit message: 基板 V2.0
Parts:
- C1, C2, R1, R2, R3: footprint BM71-Dongle:1608Metric -> BM71-Dongle:1005Metric
- SW1, SW2: footprint BM71-Dongle:SW_TVAF06 -> BM71-Dongle:SideSW_THAF01-NC-R
- moved SW1 5.07 mm to (4.33, -9.00)
- moved SW2 5.07 mm to (-4.33, -9.00), turned to 0 degrees
- moved R2 2.69 mm to (1.00, -9.10), turned to 90 degrees
- moved R3 2.69 mm to (-1.00, -9.10), turned to 90 degrees
- moved D1 2.20 mm to (0.00, -11.8), turned to 0 degrees
- moved R1 1.90 mm to (0.00, -9.10), turned to -90 degrees
- moved U2 1.85 mm to (0.00, -5.45)
- moved C2 1.81 mm to (-2.00, -5.45), turned to -90 degrees
- moved C1 1.79 mm to (2.00, -5.50), turned to 90 degrees
Routing:
- net GND: track 45.8 -> 17.7 mm, vias 5 -> 3
- net +3.3V: track 27.9 -> 15.1 mm
- net CONFIG: track 5.10 -> 14.4 mm
- net BM71_TXD: track 4.21 -> 11.8 mm, vias 1 -> 0
- net BM71_RXD: track 4.92 -> 11.4 mm, vias 0 -> 2
- net RESET: track 9.82 -> 14.2 mm
- net Net-(D1-Pad2): track 4.55 -> 2.55 mm
- net +5V: track 10.6 -> 8.78 mm
- net LED: track 8.86 -> 7.19 mm
Other:
- board size 12 x 17 mm -> 12 x 13 mm
- board text added: "BM71-Dongle V2.0"
- board text removed: "BM71-Dongle V1.0"
