File: BM71-Dongle.kicad_sch (KiCad schematic)
At the start: 11 parts, among them J1 USB_B_Micro, SW1 SW, SW2 SW, U1 BM71, U2 NJM12877F33

Commit message: 基板 V2.0
Parts:
- C1, C2, R1, R2, R3: footprint BM71-Dongle:1608Metric -> BM71-Dongle:1005Metric
- SW1, SW2: footprint BM71-Dongle:SW_TVAF06 -> BM71-Dongle:SideSW_THAF01-NC-R
Changed lines of the file:
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@@
       (effects (font (size 1.27 1.27)) hide)
     )
-    (property "Footprint" "BM71-Dongle:SW_TVAF06" (id 2) (at 212.09 90.17 0)
+    (property "Footprint" "BM71-Dongle:SideSW_THAF01-NC-R" (id 2) (at 212.09 90.17 0)
       (effects (font (size 1.27 1.27)) hide)
     )
@@
       (effects (font (size 1.016 1.016)) hide)
     )
-    (property "Footprint" "BM71-Dongle:1608Metric" (id 2) (at 212.09 64.77 0)
+    (property "Footprint" "BM71-Dongle:1005Metric" (id 2) (at 212.09 64.77 0)
       (effects (font (size 1.27 1.27)) hide)
     )
@@
       (effects (font (size 1.27 1.27)) (justify left))
     )
-    (property "Footprint" "BM71-Dongle:1608Metric" (id 2) (at 91.44 101.6 0)
+    (property "Footprint" "BM71-Dongle:1005Metric" (id 2) (at 91.44 101.6 0)
       (effects (font (size 1.27 1.27)) hide)
     )
@@
       (effects (font (size 1.016 1.016)))
     )
-    (property "Footprint" "BM71-Dongle:1608Metric" (id 2) (at 204.47 92.71 0)
+    (property "Footprint" "BM71-Dongle:1005Metric" (id 2) (at 204.47 92.71 0)
       (effects (font (size 1.27 1.27)) hide)
     )
@@
       (effects (font (size 1.27 1.27)) hide)
     )
-    (property "Footprint" "BM71-Dongle:SW_TVAF06" (id 2) (at 212.09 74.93 0)
+    (property "Footprint" "BM71-Dongle:SideSW_THAF01-NC-R" (id 2) (at 212.09 74.93 0)
       (effects (font (size 1.27 1.27)) hide)
     )
@@
       (effects (font (size 1.016 1.016)))
     )
-    (property "Footprint" "BM71-Dongle:1608Metric" (id 2) (at 204.47 77.47 0)
+    (property "Footprint" "BM71-Dongle:1005Metric" (id 2) (at 204.47 77.47 0)
       (effects (font (size 1.27 1.27)) hide)
     )
@@
       (effects (font (size 1.27 1.27)) (justify right))
     )
-    (property "Footprint" "BM71-Dongle:1608Metric" (id 2) (at 66.04 101.6 0)
+    (property "Footprint" "BM71-Dongle:1005Metric" (id 2) (at 66.04 101.6 0)
       (effects (font (size 1.27 1.27)) hide)
     )
@@
     )
     (path "/e98e30c7-cb8c-4098-8fa1-896d9d4d467f"
-      (reference "C1") (unit 1) (value "1uF") (footprint "BM71-Dongle:1608Metric")
+      (reference "C1") (unit 1) (value "1uF") (footprint "BM71-Dongle:1005Metric")
     )
     (path "/6a60c8a1-b165-4c32-a688-f2b180b5d56a"
-      (reference "C2") (unit 1) (value "1uF") (footprint "BM71-Dongle:1608Metric")
+      (reference "C2") (unit 1) (value "1uF") (footprint "BM71-Dongle:1005Metric")
     )
     (path "/80b306bb-0758-46ff-aeeb-e993e37c6eec"
@@
     )
     (path "/3cb79714-3333-4ffd-ba62-1d2c2b9890f3"
-      (reference "R1") (unit 1) (value "R") (footprint "BM71-Dongle:1608Metric")
+      (reference "R1") (unit 1) (value "R") (footprint "BM71-Dongle:1005Metric")
     )
     (path "/b062d127-92eb-472c-aae7-2a1b11d5a100"
-      (reference "R2") (unit 1) (value "4k7") (footprint "BM71-Dongle:1608Metric")
+      (reference "R2") (unit 1) (value "4k7") (footprint "BM71-Dongle:1005Metric")
     )
     (path "/a114ed5e-485b-48e6-912b-df7541100e3a"
-      (reference "R3") (unit 1) (value "4k7") (footprint "BM71-Dongle:1608Metric")
+      (reference "R3") (unit 1) (value "4k7") (footprint "BM71-Dongle:1005Metric")
     )
     (path "/aa34877d-1fa8-4889-9122-d93831301121"
-      (reference "SW1") (unit 1) (value "SW") (footprint "BM71-Dongle:SW_TVAF06")
+      (reference "SW1") (unit 1) (value "SW") (footprint "BM71-Dongle:SideSW_THAF01-NC-R")
     )
     (path "/0afcb3db-44eb-491e-93a3-f4f09a4ab0b1"
-      (reference "SW2") (unit 1) (value "SW") (footprint "BM71-Dongle:SW_TVAF06")
+      (reference "SW2") (unit 1) (value "SW") (footprint "BM71-Dongle:SideSW_THAF01-NC-R")
     )
     (path "/e991525a-0960-4dac-848d-1269493b3885"
